File: Electronics/amigoscope/amigoscope.kicad_pcb (KiCad board)
At the start: 2 copper layers, 100 x 50 mm, 21 parts, among them J1 USB_C_Receptacle_USB2.0_14P, J2 Probes, SW1 RST, SW2 BOOT, U1 ESP32-S3-WROOM-1, U2 NCP1117-3.3_SOT223, U3 TVS1400DRV, U4 MAX11612

Commit message: finished pcb
Parts:
- moved J2 206.8 mm to (143.7, 109.2)
- moved SSD1306 189.3 mm to (141.8, 67.5), turned to 90 degrees
- moved U4 177.8 mm to (148.9, 99.6), turned to 90 degrees
- moved R6 166.8 mm to (151.4, 97.9), turned to -90 degrees
- moved C3 165.1 mm to (144.5, 98.1), turned to -90 degrees
- moved R5 162.2 mm to (146.4, 97.9), turned to -90 degrees
- moved R3 142.7 mm to (126.2, 95.0), turned to 90 degrees
- moved R4 141.7 mm to (126.2, 91.8), turned to -90 degrees
- moved SW2 134.3 mm to (113.9, 74.9)
- moved C2 134.1 mm to (117.7, 74.8), turned to 90 degrees
- moved R2 133.6 mm to (119.5, 74.6), turned to -90 degrees
- moved C1 133.2 mm to (106.0, 103.1), turned to -90 degrees
- moved SW1 130.1 mm to (109.9, 103.0), turned to 180 degrees
- moved C4 129.8 mm to (105.2, 105.8)
- moved R1 125.0 mm to (104.3, 103.3), turned to 90 degrees
Routing:
- net +3V3: track 9.13 -> 130.0 mm, vias 0 -> 3
- net /SCL: track 0.00 -> 60.3 mm, vias 0 -> 2
- net /SDA: track 0.00 -> 59.3 mm
- net Net-(U1-EN): track 0.00 -> 13.8 mm
- net Net-(U1-IO0): track 0.00 -> 13.4 mm
- net /X_{2}: track 0.00 -> 12.5 mm
- net /X_{1}: track 0.00 -> 12.4 mm
- net /V_{REF}: track 0.00 -> 9.30 mm
- net /X_{0}: track 0.00 -> 9.24 mm
- net Net-(U2-VI): track 16.8 -> 19.5 mm
- net GND: track 0.00 -> 1.65 mm, vias 0 -> 2
- added copper zone on F.Cu, net GND
Other:
- board size 100 x 50 mm -> 75 x 50 mm
